File: hardware/power_board_for_egs002/power_board_for_egs002.sch (KiCad schematic (older format))
At the start: 5 parts, among them J01 +HV, J02 +12V, J03 +5V, J04 MODULATION_OUT

Commit message: continue sch update
Parts:
- removed J04: MODULATION_OUT, symbol Connector_Generic:Conn_01x02
- added J04: BRIGDE_OUT_2, symbol Connector_Generic:Conn_01x01
- added J05: BRIGDE_OUT_1, symbol Connector_Generic:Conn_01x01
- added J06: HV_SENSE, symbol Connector_Generic:Conn_01x02
- gave numbers to parts that had none: 1
Connections:
- net PowerBoard/BRIDGE_OUT_1: now also J05.1 (Pin_1)
- net PowerBoard/BRIDGE_OUT_2: now also J04.1 (Pin_1)
- net PowerSupply/+5V_OUT renamed PowerBoard/NTC_5V
- new net PowerBoard/HV_SENSE_L: J06.1 (Pin_1)
- new net PowerBoard/HV_SENSE_N: J06.2 (Pin_2)
Other:
- note added: "Notice:\nBRIDGE_OUT_2 is LIVE\nBRIDGE_OUT_1 is NEUTRAL"
Changed lines of the file:
@@
 $EndSheet
 $Sheet
-S 6200 1700 1150 1450
+S 6200 1400 1150 1750
 U 61AF7571
 F0 "PowerBoard" 50
@@
 F12 "BRIDGE_OUT_2" O R 7350 2300 50
 F13 "BRIDGE_OUT_1" O R 7350 2400 50
-F14 "HV_SENSE_A" I R 7350 1800 50
-F15 "HV_SENSE_B" I R 7350 1900 50
+F14 "HV_IN" I L 6200 1500 50
+F15 "NTC_5V" I L 6200 1600 50
+F16 "HV_SENSE_L" I R 7350 1500 50
+F17 "HV_SENSE_N" I R 7350 1600 50
 $EndSheet
 $Comp
-L power_board_for_egs002:EGS002 U?
+L power_board_for_egs002:EGS002 U01
 U 1 1 61AF7641
 P 4750 1800
-F 0 "U?" H 5100 2065 50  0000 C CNN
+F 0 "U01" H 5100 2065 50  0000 C CNN
 F 1 "EGS002" H 5100 1974 50  0000 C CNN
 F 2 "" H 4950 450 50  0001 C CNN
@@
 Wire Wire Line
 	6200 3000 5550 3000
-$Comp
-L Connector_Generic:Conn_01x02 J04
-U 1 1 61B678D0
-P 8650 2300
-F 0 "J04" H 8730 2292 50  0000 L CNN
-F 1 "MODULATION_OUT" H 8730 2201 50  0000 L CNN
-F 2 "" H 8650 2300 50  0001 C CNN
-F 3 "~" H 8650 2300 50  0001 C CNN
-	1    8650 2300
-	1    0    0    -1
-$EndComp
 Wire Wire Line
 	7350 2300 8450 2300
 Wire Wire Line
 	7350 2400 8450 2400
+Wire Wire Line
+	3950 1350 6050 1350
+Wire Wire Line
+	6050 1350 6050 1500
+Wire Wire Line
+	6050 1500 6200 1500
+Wire Wire Line
+	4100 1550 4300 1550
+Wire Wire Line
+	4300 1550 4300 1450
+Wire Wire Line
+	4300 1450 5950 1450
+Wire Wire Line
+	5950 1450 5950 1600
+Wire Wire Line
+	5950 1600 6200 1600
+Connection ~ 4100 1550
+Text Notes 7500 2700 0    50   ~ 0
+Notice:\nBRIDGE_OUT_2 is LIVE\nBRIDGE_OUT_1 is NEUTRAL
+$Comp
+L Connector_Generic:Conn_01x01 J04
+U 1 1 62CDE1E0
+P 8850 2250
+F 0 "J04" H 8930 2292 50  0000 L CNN
+F 1 "BRIGDE_OUT_2" H 8930 2201 50  0000 L CNN
+F 2 "" H 8850 2250 50  0001 C CNN
+F 3 "~" H 8850 2250 50  0001 C CNN
+	1    8850 2250
+	1    0    0    -1
+$EndComp
+$Comp
+L Connector_Generic:Conn_01x01 J05
+U 1 1 62CDE649
+P 8850 2450
+F 0 "J05" H 8930 2492 50  0000 L CNN
+F 1 "BRIGDE_OUT_1" H 8930 2401 50  0000 L CNN
+F 2 "" H 8850 2450 50  0001 C CNN
+F 3 "~" H 8850 2450 50  0001 C CNN
+	1    8850 2450
+	1    0    0    -1
+$EndComp
+Wire Wire Line
+	8450 2300 8450 2250
+Wire Wire Line
+	8450 2250 8650 2250
+Wire Wire Line
+	8650 2450 8450 2450
+Wire Wire Line
+	8450 2450 8450 2400
+$Comp
+L Connector_Generic:Conn_01x02 J06
+U 1 1 62CE110A
+P 8850 1500
+F 0 "J06" H 8930 1492 50  0000 L CNN
+F 1 "HV_SENSE" H 8930 1401 50  0000 L CNN
+F 2 "" H 8850 1500 50  0001 C CNN
+F 3 "~" H 8850 1500 50  0001 C CNN
+	1    8850 1500
+	1    0    0    -1
+$EndComp
+Wire Wire Line
+	8650 1500 7350 1500
+Wire Wire Line
+	7350 1600 8650 1600
 $EndSCHEMATC

Commit message: start adding footprints
Parts:
- added U?: SK68-100SA, power_board_for_egs002:SK68-100SA, symbol power_board_for_egs002:SK68-100SA
- U01: footprint (none) -> power_board_for_egs002:EGS002
Connections:
- net GND: now also U?.1 (P1), U?.2 (P2), U?.3 (P3), U?.4 (P4)
Changed lines of the file:
@@
 F 0 "U01" H 5100 2065 50  0000 C CNN
 F 1 "EGS002" H 5100 1974 50  0000 C CNN
-F 2 "" H 4950 450 50  0001 C CNN
+F 2 "power_board_for_egs002:EGS002" H 4950 450 50  0001 C CNN
 F 3 "" H 4950 450 50  0001 C CNN
 	1    4750 1800
@@
 Wire Wire Line
 	7350 1600 8650 1600
+$Comp
+L power_board_for_egs002:SK68-100SA U?
+U 1 1 61B3967E
+P 10400 650
+F 0 "U?" H 10628 546 50  0000 L CNN
+F 1 "SK68-100SA" H 10628 455 50  0000 L CNN
+F 2 "power_board_for_egs002:SK68-100SA" H 10400 650 50  0001 C CNN
+F 3 "" H 10400 650 50  0001 C CNN
+	1    10400 650
+	1    0    0    -1
+$EndComp
+$Comp
+L power:GND #PWR?
+U 1 1 61B39DC2
+P 10200 1050
+F 0 "#PWR?" H 10200 800 50  0001 C CNN
+F 1 "GND" H 10205 877 50  0000 C CNN
+F 2 "" H 10200 1050 50  0001 C CNN
+F 3 "" H 10200 1050 50  0001 C CNN
+	1    10200 1050
+	1    0    0    -1
+$EndComp
+Wire Wire Line
+	10200 1050 10200 950
+Wire Wire Line
+	10200 650  10300 650
+Wire Wire Line
+	10300 750  10200 750
+Connection ~ 10200 750
+Wire Wire Line
+	10200 750  10200 650
+Wire Wire Line
+	10300 850  10200 850
+Connection ~ 10200 850
+Wire Wire Line
+	10200 850  10200 750
+Wire Wire Line
+	10300 950  10200 950
+Connection ~ 10200 950
+Wire Wire Line
+	10200 950  10200 850
 $EndSCHEMATC

Commit message: continue sch dev
Parts:
- removed J04: BRIGDE_OUT_2, symbol Connector_Generic:Conn_01x01
- removed J05: BRIGDE_OUT_1, symbol Connector_Generic:Conn_01x01
- added J4: BRIGDE_OUT_2, power_board_for_egs002:conn_5.08, symbol Connector_Generic:Conn_01x02
- added J5: BRIGDE_OUT_1, power_board_for_egs002:conn_5.08, symbol Connector_Generic:Conn_01x02
- J1: renamed from J01; footprint (none) -> power_board_for_egs002:conn_5.08
- J2: renamed from J02; footprint (none) -> power_board_for_egs002:conn_5.08
- J3: renamed from J03; footprint (none) -> power_board_for_egs002:conn_2.54
- J6: renamed from J06; footprint (none) -> power_board_for_egs002:conn_2.54
- gave numbers to parts that had none: 1
- renumbered U01 to U1
Connections:
- net PowerBoard/BRIDGE_OUT_1: now also J5.1 (Pin_1), J5.2 (Pin_2)
- net PowerBoard/BRIDGE_OUT_2: now also J4.1 (Pin_1), J4.2 (Pin_2)
Changed lines of the file:
@@
 $EndSheet
 $Comp
-L power_board_for_egs002:EGS002 U01
+L power_board_for_egs002:EGS002 U1
 U 1 1 61AF7641
 P 4750 1800
-F 0 "U01" H 5100 2065 50  0000 C CNN
+F 0 "U1" H 5100 2065 50  0000 C CNN
 F 1 "EGS002" H 5100 1974 50  0000 C CNN
 F 2 "power_board_for_egs002:EGS002" H 4950 450 50  0001 C CNN
@@
 $EndComp
 $Comp
-L Connector_Generic:Conn_01x02 J01
+L Connector_Generic:Conn_01x02 J1
 U 1 1 61B554F8
 P 850 950
-F 0 "J01" H 768 1167 50  0000 C CNN
+F 0 "J1" H 768 1167 50  0000 C CNN
 F 1 "+HV" H 768 1076 50  0000 C CNN
-F 2 "" H 850 950 50  0001 C CNN
+F 2 "power_board_for_egs002:conn_5.08" H 850 950 50  0001 C CNN
 F 3 "~" H 850 950 50  0001 C CNN
 	1    850  950
@@
 $EndComp
 $Comp
-L Connector_Generic:Conn_01x02 J02
+L Connector_Generic:Conn_01x02 J2
 U 1 1 61B55BA7
 P 850 1750
-F 0 "J02" H 768 1967 50  0000 C CNN
+F 0 "J2" H 768 1967 50  0000 C CNN
 F 1 "+12V" H 768 1876 50  0000 C CNN
-F 2 "" H 850 1750 50  0001 C CNN
+F 2 "power_board_for_egs002:conn_5.08" H 850 1750 50  0001 C CNN
 F 3 "~" H 850 1750 50  0001 C CNN
 	1    850  1750
@@
 $EndComp
 $Comp
-L Connector_Generic:Conn_01x02 J03
+L Connector_Generic:Conn_01x02 J3
 U 1 1 61B55DD1
 P 850 2600
-F 0 "J03" H 768 2817 50  0000 C CNN
+F 0 "J3" H 768 2817 50  0000 C CNN
 F 1 "+5V" H 768 2726 50  0000 C CNN
-F 2 "" H 850 2600 50  0001 C CNN
+F 2 "power_board_for_egs002:conn_2.54" H 850 2600 50  0001 C CNN
 F 3 "~" H 850 2600 50  0001 C CNN
 	1    850  2600
@@
 $EndComp
 $Comp
-L power:GND #PWR?
+L power:GND #PWR0101
 U 1 1 61B5629D
 P 1100 1100
-F 0 "#PWR?" H 1100 850 50  0001 C CNN
+F 0 "#PWR0101" H 1100 850 50  0001 C CNN
 F 1 "GND" H 1105 927 50  0000 C CNN
 F 2 "" H 1100 1100 50  0001 C CNN
@@
 	1100 1050 1100 1100
 $Comp
-L power:GND #PWR?
+L power:GND #PWR0102
 U 1 1 61B56F10
 P 1100 1900
-F 0 "#PWR?" H 1100 1650 50  0001 C CNN
+F 0 "#PWR0102" H 1100 1650 50  0001 C CNN
 F 1 "GND" H 1105 1727 50  0000 C CNN
 F 2 "" H 1100 1900 50  0001 C CNN
@@
 $EndComp
 $Comp
-L power:GND #PWR?
+L power:GND #PWR0103
 U 1 1 61B5849A
 P 1100 2750
-F 0 "#PWR?" H 1100 2500 50  0001 C CNN
+F 0 "#PWR0103" H 1100 2500 50  0001 C CNN
 F 1 "GND" H 1105 2577 50  0000 C CNN
 F 2 "" H 1100 2750 50  0001 C CNN
@@
 	1100 2700 1100 2750
 $Comp
-L power:GND #PWR?
+L power:GND #PWR0104
 U 1 1 61B5B492
 P 4550 2950
-F 0 "#PWR?" H 4550 2700 50  0001 C CNN
+F 0 "#PWR0104" H 4550 2700 50  0001 C CNN
 F 1 "GND" H 4555 2777 50  0000 C CNN
 F 2 "" H 4550 2950 50  0001 C CNN
@@
 Text Notes 7500 2700 0    50   ~ 0
 Notice:\nBRIDGE_OUT_2 is LIVE\nBRIDGE_OUT_1 is NEUTRAL
-$Comp
-L Connector_Generic:Conn_01x01 J04
-U 1 1 62CDE1E0
-P 8850 2250
-F 0 "J04" H 8930 2292 50  0000 L CNN
-F 1 "BRIGDE_OUT_2" H 8930 2201 50  0000 L CNN
-F 2 "" H 8850 2250 50  0001 C CNN
-F 3 "~" H 8850 2250 50  0001 C CNN
-	1    8850 2250
-	1    0    0    -1
-$EndComp
-$Comp
-L Connector_Generic:Conn_01x01 J05
-U 1 1 62CDE649
-P 8850 2450
-F 0 "J05" H 8930 2492 50  0000 L CNN
-F 1 "BRIGDE_OUT_1" H 8930 2401 50  0000 L CNN
-F 2 "" H 8850 2450 50  0001 C CNN
-F 3 "~" H 8850 2450 50  0001 C CNN
-	1    8850 2450
-	1    0    0    -1
-$EndComp
 Wire Wire Line
 	8450 2300 8450 2250
@@
 	8450 2450 8450 2400
 $Comp
-L Connector_Generic:Conn_01x02 J06
+L Connector_Generic:Conn_01x02 J6
 U 1 1 62CE110A
 P 8850 1500
-F 0 "J06" H 8930 1492 50  0000 L CNN
+F 0 "J6" H 8930 1492 50  0000 L CNN
 F 1 "HV_SENSE" H 8930 1401 50  0000 L CNN
-F 2 "" H 8850 1500 50  0001 C CNN
+F 2 "power_board_for_egs002:conn_2.54" H 8850 1500 50  0001 C CNN
 F 3 "~" H 8850 1500 50  0001 C CNN
 	1    8850 1500
@@
 	7350 1600 8650 1600
 $Comp
-L power_board_for_egs002:SK68-100SA U?
+L power_board_for_egs002:SK68-100SA U2
 U 1 1 61B3967E
 P 10400 650
-F 0 "U?" H 10628 546 50  0000 L CNN
+F 0 "U2" H 10628 546 50  0000 L CNN
 F 1 "SK68-100SA" H 10628 455 50  0000 L CNN
 F 2 "power_board_for_egs002:SK68-100SA" H 10400 650 50  0001 C CNN
@@
 $EndComp
 $Comp
-L power:GND #PWR?
+L power:GND #PWR0105
 U 1 1 61B39DC2
 P 10200 1050
-F 0 "#PWR?" H 10200 800 50  0001 C CNN
+F 0 "#PWR0105" H 10200 800 50  0001 C CNN
 F 1 "GND" H 10205 877 50  0000 C CNN
 F 2 "" H 10200 1050 50  0001 C CNN
@@
 Wire Wire Line
 	10200 950  10200 850
+$Comp
+L Connector_Generic:Conn_01x02 J4
+U 1 1 61B47699
+P 8850 2150
+F 0 "J4" H 8930 2142 50  0000 L CNN
+F 1 "BRIGDE_OUT_2" H 8930 2051 50  0000 L CNN
+F 2 "power_board_for_egs002:conn_5.08" H 8850 2150 50  0001 C CNN
+F 3 "~" H 8850 2150 50  0001 C CNN
+	1    8850 2150
+	1    0    0    -1
+$EndComp
+$Comp
+L Connector_Generic:Conn_01x02 J5
+U 1 1 61B47860
+P 8850 2450
+F 0 "J5" H 8930 2442 50  0000 L CNN
+F 1 "BRIGDE_OUT_1" H 8930 2351 50  0000 L CNN
+F 2 "power_board_for_egs002:conn_5.08" H 8850 2450 50  0001 C CNN
+F 3 "~" H 8850 2450 50  0001 C CNN
+	1    8850 2450
+	1    0    0    -1
+$EndComp
+Wire Wire Line
+	8650 2150 8450 2150
+Wire Wire Line
+	8450 2150 8450 2250
+Connection ~ 8450 2250
+Wire Wire Line
+	8650 2550 8450 2550
+Wire Wire Line
+	8450 2550 8450 2450
+Connection ~ 8450 2450
 $EndSCHEMATC
