File: hardware/power_board_for_egs002/powerBoard.sch (KiCad schematic (older format))
At the start: 0 parts

Commit message: continue sch update
Parts:
- added C21, C22, C25: 100n, Capacitor_SMD:C_1206_3216Metric, symbol Device:C_Small
- added C23, C26: 100n, symbol Device:C_Small
- added C24: 4.7u, symbol Device:C_Small
- added D21, D210, D211, D212, D22, D23, D24, D25, D26, D27, D28, D29: 1N4148, Diode_THT:D_DO-35_SOD27_P7.62mm_Horizontal, symbol Diode:1N4148
- added D213, D214, D215, D216: 1N4007, Diode_THT:D_DO-41_SOD81_P10.16mm_Horizontal, symbol Diode:1N4007
- added J21, J23: Conn_01x02, symbol Connector_Generic:Conn_01x02
- added J22: Conn_01x03, Connector_PinHeader_2.54mm:PinHeader_1x03_P2.54mm_Vertical, symbol Connector_Generic:Conn_01x03
- added J24: HV_SENSE_SELECT_A, Connector_PinHeader_2.54mm:PinHeader_1x03_P2.54mm_Vertical, symbol Connector_Generic:Conn_01x03
- added J25: HV_SENSE_SELECT_B, Connector_PinHeader_2.54mm:PinHeader_1x03_P2.54mm_Vertical, symbol Connector_Generic:Conn_01x03
- added J26: Conn_01x02, Connector_PinHeader_2.54mm:PinHeader_1x02_P2.54mm_Vertical, symbol Connector_Generic:Conn_01x02
- added Q21, Q22, Q23, Q24, Q25, Q26, Q27, Q28: TK40E06N1, Package_TO_SOT_THT:TO-220-3_Vertical, symbol Device:Q_NMOS_GDS
- added R21, R211, R213, R215, R23, R25, R27, R29: 5.6, Resistor_SMD:R_1206_3216Metric, symbol Device:R_Small
- added R210, R212, R214, R216, R217, R218, R219, R22, R220, R24, R26, R28: 10k, Resistor_SMD:R_1206_3216Metric, symbol Device:R_Small
- added R217: R_Small, Resistor_SMD:R_1206_3216Metric, symbol Device:R_Small
- added R221, R222, R223, R224, R225, R226, R227, R228, R229, R230, R231, R232: 33k, symbol Device:R_Small
- added R227, R233: 10k, symbol Device:R_Small
- added RV21, RV22, RV23: 100k, Connector_PinHeader_2.54mm:PinHeader_1x03_P2.54mm_Vertical, symbol Device:R_POT
Connections:
- net 1_HO: now also D25.1 (K), D27.1 (K), R213.1, R29.1
- net 1_LO: now also D26.1 (K), D28.1 (K), R211.1, R215.1
- net 1_VS: now also Q25.3 (S), Q26.2 (D), Q27.3 (S), Q28.2 (D), R210.1, R214.1
- net 2_HO: now also D21.1 (K), D23.1 (K), R21.2, R25.2
- net 2_LO: now also D22.1 (K), D24.1 (K), R23.2, R27.2
- net 2_VS: now also Q21.3 (S), Q22.2 (D), Q23.3 (S), Q24.2 (D), R22.1, R26.1
- net I_FB: now also J22.2 (Pin_2)
- net T_FB: now also C26.1, J26.2 (Pin_2)
- net V_FB: now also C22.1, J25.2 (Pin_2)
- new net: D21.2 (A), Q21.1 (G), R21.1, R22.2
- new net: D23.2 (A), Q23.1 (G), R25.1, R26.2
- new net: D22.2 (A), Q22.1 (G), R23.1, R24.2
- new net: J21.1 (Pin_1), J22.1 (Pin_1), Q22.3 (S), Q24.3 (S), Q26.3 (S), Q28.3 (S), R212.1, R216.1, R217.1, R24.1, R28.1
- new net: D24.2 (A), Q24.1 (G), R27.1, R28.2
- new net: D27.2 (A), Q27.1 (G), R213.2, R214.2
- new net: D25.2 (A), Q25.1 (G), R210.2, R29.2
- new net: D26.2 (A), Q26.1 (G), R211.2, R212.2
- new net: D28.2 (A), Q28.1 (G), R215.2, R216.2
- new net: R221.1, R222.2
- new net: J24.1 (Pin_1), R221.2
- new net: R226.1, R227.2, RV22.1
- new net: C21.1, J25.1 (Pin_1), RV22.2
- new net: D213.1 (K), D214.1 (K), R227.2
- new net: D213.2 (A), D215.1 (K), J24.3 (Pin_3)
- new net: D215.2 (A), D216.2 (A), R230.2
- new net: R227.1, R228.2
- new net: R222.1, R223.2
- new net: R223.1, R224.2
- new net: R224.1, R225.2
- new net: R225.1, R226.2
- new net: R228.1, R229.2
- new net: R229.1, R233.2, RV23.1
- new net: R230.1, R231.2
- new net: R231.1, R232.2
- new net: C23.1, C24.1, J25.3 (Pin_3), RV23.2
- new net: D210.1 (K), D29.2 (A), J23.1 (Pin_1)
- new net: D211.2 (A), D212.1 (K), J23.2 (Pin_2)
- new net: D211.1 (K), D29.1 (K), R217.2, R218.2, R219.2, R220.2, RV21.1
- new net: C25.1, J22.3 (Pin_3), RV21.2
- new net GND: C21.2, C22.2, C23.2, C24.2, C25.2, C26.2, D210.2 (A), D212.2 (A), J21.2 (Pin_2), R217.1, R217.2, R218.1, R219.1, R220.1, R227.1, R232.1, R233.1, RV21.3, RV22.3, RV23.3
- new net HV_IN: Q21.2 (D), Q23.2 (D), Q25.2 (D), Q27.2 (D)
- new net HV_SENSE_L: J24.2 (Pin_2)
- new net HV_SENSE_N: D214.2 (A), D216.1 (K)
- new net NTC_5V: J26.1 (Pin_1)

Commit message: start adding footprints
Parts:
- C23, C26: footprint (none) -> Capacitor_SMD:C_1206_3216Metric
- C24: footprint (none) -> Capacitor_THT:CP_Radial_D5.0mm_P2.50mm
- D21, D210, D211, D212, D22, D23, D24, D25, D26, D27, D28, D29: footprint Diode_THT:D_DO-35_SOD27_P7.62mm_Horizontal -> Diode_THT:D_DO-35_SOD27_P2.54mm_Vertical_AnodeUp
- D213, D214, D215, D216: footprint Diode_THT:D_DO-41_SOD81_P10.16mm_Horizontal -> Diode_THT:D_DO-41_SOD81_P5.08mm_Vertical_AnodeUp
- R221, R222, R223, R224, R225, R226, R227, R228, R229, R230, R231, R232, R233: footprint (none) -> Resistor_SMD:R_1206_3216Metric
Changed lines of the file:
@@
 F 0 "D21" V 1604 1329 50  0000 L CNN
 F 1 "1N4148" V 1695 1329 50  0000 L CNN
-F 2 "Diode_THT:D_DO-35_SOD27_P7.62mm_Horizontal" H 1650 1075 50  0001 C CNN
+F 2 "Diode_THT:D_DO-35_SOD27_P2.54mm_Vertical_AnodeUp" H 1650 1075 50  0001 C CNN
 F 3 "https://assets.nexperia.com/documents/data-sheet/1N4148_1N4448.pdf" H 1650 1250 50  0001 C CNN
 	1    1650 1250
@@
 F 0 "D23" V 3004 1329 50  0000 L CNN
 F 1 "1N4148" V 3095 1329 50  0000 L CNN
-F 2 "Diode_THT:D_DO-35_SOD27_P7.62mm_Horizontal" H 3050 1075 50  0001 C CNN
+F 2 "Diode_THT:D_DO-35_SOD27_P2.54mm_Vertical_AnodeUp" H 3050 1075 50  0001 C CNN
 F 3 "https://assets.nexperia.com/documents/data-sheet/1N4148_1N4448.pdf" H 3050 1250 50  0001 C CNN
 	1    3050 1250
@@
 F 0 "D24" V 3004 2429 50  0000 L CNN
 F 1 "1N4148" V 3095 2429 50  0000 L CNN
-F 2 "Diode_THT:D_DO-35_SOD27_P7.62mm_Horizontal" H 3050 2175 50  0001 C CNN
+F 2 "Diode_THT:D_DO-35_SOD27_P2.54mm_Vertical_AnodeUp" H 3050 2175 50  0001 C CNN
 F 3 "https://assets.nexperia.com/documents/data-sheet/1N4148_1N4448.pdf" H 3050 2350 50  0001 C CNN
 	1    3050 2350
@@
 F 0 "D22" V 1604 2429 50  0000 L CNN
 F 1 "1N4148" V 1695 2429 50  0000 L CNN
-F 2 "Diode_THT:D_DO-35_SOD27_P7.62mm_Horizontal" H 1650 2175 50  0001 C CNN
+F 2 "Diode_THT:D_DO-35_SOD27_P2.54mm_Vertical_AnodeUp" H 1650 2175 50  0001 C CNN
 F 3 "https://assets.nexperia.com/documents/data-sheet/1N4148_1N4448.pdf" H 1650 2350 50  0001 C CNN
 	1    1650 2350
@@
 F 0 "D28" V 14450 2550 50  0000 R CNN
 F 1 "1N4148" V 14550 2700 50  0000 R CNN
-F 2 "Diode_THT:D_DO-35_SOD27_P7.62mm_Horizontal" H 14650 2175 50  0001 C CNN
+F 2 "Diode_THT:D_DO-35_SOD27_P2.54mm_Vertical_AnodeUp" H 14650 2175 50  0001 C CNN
 F 3 "https://assets.nexperia.com/documents/data-sheet/1N4148_1N4448.pdf" H 14650 2350 50  0001 C CNN
 	1    14650 2350
@@
 F 0 "D27" V 14450 1450 50  0000 R CNN
 F 1 "1N4148" V 14550 1600 50  0000 R CNN
-F 2 "Diode_THT:D_DO-35_SOD27_P7.62mm_Horizontal" H 14650 1075 50  0001 C CNN
+F 2 "Diode_THT:D_DO-35_SOD27_P2.54mm_Vertical_AnodeUp" H 14650 1075 50  0001 C CNN
 F 3 "https://assets.nexperia.com/documents/data-sheet/1N4148_1N4448.pdf" H 14650 1250 50  0001 C CNN
 	1    14650 1250
@@
 F 0 "R221" V 3304 6350 50  0000 C CNN
 F 1 "33k" V 3395 6350 50  0000 C CNN
-F 2 "" H 3500 6350 50  0001 C CNN
+F 2 "Resistor_SMD:R_1206_3216Metric" H 3500 6350 50  0001 C CNN
 F 3 "~" H 3500 6350 50  0001 C CNN
 	1    3500 6350
@@
 F 0 "R227" H 5291 6604 50  0000 R CNN
 F 1 "10k" H 5291 6695 50  0000 R CNN
-F 2 "" H 5350 6650 50  0001 C CNN
+F 2 "Resistor_SMD:R_1206_3216Metric" H 5350 6650 50  0001 C CNN
 F 3 "~" H 5350 6650 50  0001 C CNN
 	1    5350 6650
@@
 F 0 "D213" V 2446 8521 50  0000 R CNN
 F 1 "1N4007" V 2355 8521 50  0000 R CNN
-F 2 "Diode_THT:D_DO-41_SOD81_P10.16mm_Horizontal" H 2400 8425 50  0001 C CNN
+F 2 "Diode_THT:D_DO-41_SOD81_P5.08mm_Vertical_AnodeUp" H 2400 8425 50  0001 C CNN
 F 3 "http://www.vishay.com/docs/88503/1n4001.pdf" H 2400 8600 50  0001 C CNN
 	1    2400 8600
@@
 F 0 "D214" V 2354 9179 50  0000 L CNN
 F 1 "1N4007" V 2445 9179 50  0000 L CNN
-F 2 "Diode_THT:D_DO-41_SOD81_P10.16mm_Horizontal" H 2400 8925 50  0001 C CNN
+F 2 "Diode_THT:D_DO-41_SOD81_P5.08mm_Vertical_AnodeUp" H 2400 8925 50  0001 C CNN
 F 3 "http://www.vishay.com/docs/88503/1n4001.pdf" H 2400 9100 50  0001 C CNN
 	1    2400 9100
@@
 F 0 "D216" V 3096 9021 50  0000 R CNN
 F 1 "1N4007" V 3005 9021 50  0000 R CNN
-F 2 "Diode_THT:D_DO-41_SOD81_P10.16mm_Horizontal" H 3050 8925 50  0001 C CNN
+F 2 "Diode_THT:D_DO-41_SOD81_P5.08mm_Vertical_AnodeUp" H 3050 8925 50  0001 C CNN
 F 3 "http://www.vishay.com/docs/88503/1n4001.pdf" H 3050 9100 50  0001 C CNN
 	1    3050 9100
@@
 F 0 "D215" V 3004 8679 50  0000 L CNN
 F 1 "1N4007" V 3095 8679 50  0000 L CNN
-F 2 "Diode_THT:D_DO-41_SOD81_P10.16mm_Horizontal" H 3050 8425 50  0001 C CNN
+F 2 "Diode_THT:D_DO-41_SOD81_P5.08mm_Vertical_AnodeUp" H 3050 8425 50  0001 C CNN
 F 3 "http://www.vishay.com/docs/88503/1n4001.pdf" H 3050 8600 50  0001 C CNN
 	1    3050 8600
@@
 F 0 "R227" V 4054 8050 50  0000 C CNN
 F 1 "33k" V 4145 8050 50  0000 C CNN
-F 2 "" H 4250 8050 50  0001 C CNN
+F 2 "Resistor_SMD:R_1206_3216Metric" H 4250 8050 50  0001 C CNN
 F 3 "~" H 4250 8050 50  0001 C CNN
 	1    4250 8050
@@
 F 0 "R222" V 3604 6350 50  0000 C CNN
 F 1 "33k" V 3695 6350 50  0000 C CNN
-F 2 "" H 3800 6350 50  0001 C CNN
+F 2 "Resistor_SMD:R_1206_3216Metric" H 3800 6350 50  0001 C CNN
 F 3 "~" H 3800 6350 50  0001 C CNN
 	1    3800 6350
@@
 F 0 "R223" V 3904 6350 50  0000 C CNN
 F 1 "33k" V 3995 6350 50  0000 C CNN
-F 2 "" H 4100 6350 50  0001 C CNN
+F 2 "Resistor_SMD:R_1206_3216Metric" H 4100 6350 50  0001 C CNN
 F 3 "~" H 4100 6350 50  0001 C CNN
 	1    4100 6350
@@
 F 0 "R224" V 4204 6350 50  0000 C CNN
 F 1 "33k" V 4295 6350 50  0000 C CNN
-F 2 "" H 4400 6350 50  0001 C CNN
+F 2 "Resistor_SMD:R_1206_3216Metric" H 4400 6350 50  0001 C CNN
 F 3 "~" H 4400 6350 50  0001 C CNN
 	1    4400 6350
@@
 F 0 "R225" V 4504 6350 50  0000 C CNN
 F 1 "33k" V 4595 6350 50  0000 C CNN
-F 2 "" H 4700 6350 50  0001 C CNN
+F 2 "Resistor_SMD:R_1206_3216Metric" H 4700 6350 50  0001 C CNN
 F 3 "~" H 4700 6350 50  0001 C CNN
 	1    4700 6350
@@
 F 0 "R226" V 4804 6350 50  0000 C CNN
 F 1 "33k" V 4895 6350 50  0000 C CNN
-F 2 "" H 5000 6350 50  0001 C CNN
+F 2 "Resistor_SMD:R_1206_3216Metric" H 5000 6350 50  0001 C CNN
 F 3 "~" H 5000 6350 50  0001 C CNN
 	1    5000 6350
@@
 F 0 "R228" V 4354 8050 50  0000 C CNN
 F 1 "33k" V 4445 8050 50  0000 C CNN
-F 2 "" H 4550 8050 50  0001 C CNN
+F 2 "Resistor_SMD:R_1206_3216Metric" H 4550 8050 50  0001 C CNN
 F 3 "~" H 4550 8050 50  0001 C CNN
 	1    4550 8050
@@
 F 0 "R229" V 4654 8050 50  0000 C CNN
 F 1 "33k" V 4745 8050 50  0000 C CNN
-F 2 "" H 4850 8050 50  0001 C CNN
+F 2 "Resistor_SMD:R_1206_3216Metric" H 4850 8050 50  0001 C CNN
 F 3 "~" H 4850 8050 50  0001 C CNN
 	1    4850 8050
@@
 F 0 "R230" V 4054 8850 50  0000 C CNN
 F 1 "33k" V 4145 8850 50  0000 C CNN
-F 2 "" H 4250 8850 50  0001 C CNN
+F 2 "Resistor_SMD:R_1206_3216Metric" H 4250 8850 50  0001 C CNN
 F 3 "~" H 4250 8850 50  0001 C CNN
 	1    4250 8850
@@
 F 0 "R231" V 4354 8850 50  0000 C CNN
 F 1 "33k" V 4445 8850 50  0000 C CNN
-F 2 "" H 4550 8850 50  0001 C CNN
+F 2 "Resistor_SMD:R_1206_3216Metric" H 4550 8850 50  0001 C CNN
 F 3 "~" H 4550 8850 50  0001 C CNN
 	1    4550 8850
@@
 F 0 "R232" V 4654 8850 50  0000 C CNN
 F 1 "33k" V 4745 8850 50  0000 C CNN
-F 2 "" H 4850 8850 50  0001 C CNN
+F 2 "Resistor_SMD:R_1206_3216Metric" H 4850 8850 50  0001 C CNN
 F 3 "~" H 4850 8850 50  0001 C CNN
 	1    4850 8850
@@
 F 0 "C26" H 1442 10196 50  0000 L CNN
 F 1 "100n" H 1442 10105 50  0000 L CNN
-F 2 "" H 1350 10150 50  0001 C CNN
+F 2 "Capacitor_SMD:C_1206_3216Metric" H 1350 10150 50  0001 C CNN
 F 3 "~" H 1350 10150 50  0001 C CNN
 	1    1350 10150
@@
 F 0 "C23" H 6292 8746 50  0000 L CNN
 F 1 "100n" H 6292 8655 50  0000 L CNN
-F 2 "" H 6200 8700 50  0001 C CNN
+F 2 "Capacitor_SMD:C_1206_3216Metric" H 6200 8700 50  0001 C CNN
 F 3 "~" H 6200 8700 50  0001 C CNN
 	1    6200 8700
@@
 F 0 "C24" H 6742 8746 50  0000 L CNN
 F 1 "4.7u" H 6742 8655 50  0000 L CNN
-F 2 "" H 6650 8700 50  0001 C CNN
+F 2 "Capacitor_THT:CP_Radial_D5.0mm_P2.50mm" H 6650 8700 50  0001 C CNN
 F 3 "~" H 6650 8700 50  0001 C CNN
 	1    6650 8700
@@
 F 0 "D211" V 3304 4779 50  0000 L CNN
 F 1 "1N4148" V 3395 4779 50  0000 L CNN
-F 2 "Diode_THT:D_DO-35_SOD27_P7.62mm_Horizontal" H 3350 4525 50  0001 C CNN
+F 2 "Diode_THT:D_DO-35_SOD27_P2.54mm_Vertical_AnodeUp" H 3350 4525 50  0001 C CNN
 F 3 "https://assets.nexperia.com/documents/data-sheet/1N4148_1N4448.pdf" H 3350 4700 50  0001 C CNN
 	1    3350 4700
@@
 F 0 "D210" V 2804 5179 50  0000 L CNN
 F 1 "1N4148" V 2895 5179 50  0000 L CNN
-F 2 "Diode_THT:D_DO-35_SOD27_P7.62mm_Horizontal" H 2850 4925 50  0001 C CNN
+F 2 "Diode_THT:D_DO-35_SOD27_P2.54mm_Vertical_AnodeUp" H 2850 4925 50  0001 C CNN
 F 3 "https://assets.nexperia.com/documents/data-sheet/1N4148_1N4448.pdf" H 2850 5100 50  0001 C CNN
 	1    2850 5100
@@
 F 0 "D29" V 2804 4779 50  0000 L CNN
 F 1 "1N4148" V 2895 4779 50  0000 L CNN
-F 2 "Diode_THT:D_DO-35_SOD27_P7.62mm_Horizontal" H 2850 4525 50  0001 C CNN
+F 2 "Diode_THT:D_DO-35_SOD27_P2.54mm_Vertical_AnodeUp" H 2850 4525 50  0001 C CNN
 F 3 "https://assets.nexperia.com/documents/data-sheet/1N4148_1N4448.pdf" H 2850 4700 50  0001 C CNN
 	1    2850 4700
@@
 F 0 "D212" V 3304 5179 50  0000 L CNN
 F 1 "1N4148" V 3395 5179 50  0000 L CNN
-F 2 "Diode_THT:D_DO-35_SOD27_P7.62mm_Horizontal" H 3350 4925 50  0001 C CNN
+F 2 "Diode_THT:D_DO-35_SOD27_P2.54mm_Vertical_AnodeUp" H 3350 4925 50  0001 C CNN
 F 3 "https://assets.nexperia.com/documents/data-sheet/1N4148_1N4448.pdf" H 3350 5100 50  0001 C CNN
 	1    3350 5100
@@
 F 0 "D25" V 13050 1450 50  0000 R CNN
 F 1 "1N4148" V 13150 1600 50  0000 R CNN
-F 2 "Diode_THT:D_DO-35_SOD27_P7.62mm_Horizontal" H 13250 1075 50  0001 C CNN
+F 2 "Diode_THT:D_DO-35_SOD27_P2.54mm_Vertical_AnodeUp" H 13250 1075 50  0001 C CNN
 F 3 "https://assets.nexperia.com/documents/data-sheet/1N4148_1N4448.pdf" H 13250 1250 50  0001 C CNN
 	1    13250 1250
@@
 F 0 "D26" V 13050 2550 50  0000 R CNN
 F 1 "1N4148" V 13150 2700 50  0000 R CNN
-F 2 "Diode_THT:D_DO-35_SOD27_P7.62mm_Horizontal" H 13250 2175 50  0001 C CNN
+F 2 "Diode_THT:D_DO-35_SOD27_P2.54mm_Vertical_AnodeUp" H 13250 2175 50  0001 C CNN
 F 3 "https://assets.nexperia.com/documents/data-sheet/1N4148_1N4448.pdf" H 13250 2350 50  0001 C CNN
 	1    13250 2350
@@
 F 0 "R233" H 5550 8300 50  0000 R CNN
 F 1 "10k" H 5550 8350 50  0000 R CNN
-F 2 "" H 5300 8500 50  0001 C CNN
+F 2 "Resistor_SMD:R_1206_3216Metric" H 5300 8500 50  0001 C CNN
 F 3 "~" H 5300 8500 50  0001 C CNN
 	1    5300 8500

Commit message: continue sch dev
Parts:
- removed C21, C23: 100n, Capacitor_SMD:C_1206_3216Metric, symbol Device:C_Small
- J21: footprint (none) -> power_board_for_egs002:conn_5.08
- J23: footprint (none) -> power_board_for_egs002:conn_2.54
- J26: footprint Connector_PinHeader_2.54mm:PinHeader_1x02_P2.54mm_Vertical -> power_board_for_egs002:conn_2.54
- renumbered R227 to R234, R217 to R235
Changed lines of the file:
@@
 1_VS
 $Comp
-L Device:R_Small R217
+L Device:R_Small R235
 U 1 1 61D8A125
 P 2050 3550
-F 0 "R217" H 2109 3596 50  0000 L CNN
+F 0 "R235" H 2109 3596 50  0000 L CNN
 F 1 "R_Small" H 2109 3505 50  0000 L CNN
 F 2 "Resistor_SMD:R_1206_3216Metric" H 2050 3550 50  0001 C CNN
@@
 $EndComp
 $Comp
-L power:GND #PWR?
+L power:GND #PWR0115
 U 1 1 61D8DD08
 P 2050 3750
-F 0 "#PWR?" H 2050 3500 50  0001 C CNN
+F 0 "#PWR0115" H 2050 3500 50  0001 C CNN
 F 1 "GND" H 2055 3577 50  0000 C CNN
 F 2 "" H 2050 3750 50  0001 C CNN
@@
 F 0 "J26" H 1780 9892 50  0000 L CNN
 F 1 "Conn_01x02" H 1780 9801 50  0000 L CNN
-F 2 "Connector_PinHeader_2.54mm:PinHeader_1x02_P2.54mm_Vertical" H 1700 9900 50  0001 C CNN
+F 2 "power_board_for_egs002:conn_2.54" H 1700 9900 50  0001 C CNN
 F 3 "~" H 1700 9900 50  0001 C CNN
 	1    1700 9900
@@
 $EndComp
 $Comp
-L Device:R_Small R227
+L Device:R_Small R234
 U 1 1 61E6F9F8
 P 5350 6650
-F 0 "R227" H 5291 6604 50  0000 R CNN
+F 0 "R234" H 5291 6604 50  0000 R CNN
 F 1 "10k" H 5291 6695 50  0000 R CNN
 F 2 "Resistor_SMD:R_1206_3216Metric" H 5350 6650 50  0001 C CNN
@@
 Wire Wire Line
 	5900 6950 5350 6950
-$Comp
-L Device:C_Small C21
-U 1 1 61E81DD0
-P 6300 6700
-F 0 "C21" H 6392 6746 50  0000 L CNN
-F 1 "100n" H 6392 6655 50  0000 L CNN
-F 2 "Capacitor_SMD:C_1206_3216Metric" H 6300 6700 50  0001 C CNN
-F 3 "~" H 6300 6700 50  0001 C CNN
-	1    6300 6700
-	1    0    0    -1
-$EndComp
 Wire Wire Line
 	6300 6600 6300 6350
@@
 Connection ~ 5900 6950
 $Comp
-L power:GND #PWR?
+L power:GND #PWR0116
 U 1 1 61E9524F
 P 5900 7050
-F 0 "#PWR?" H 5900 6800 50  0001 C CNN
+F 0 "#PWR0116" H 5900 6800 50  0001 C CNN
 F 1 "GND" H 5905 6877 50  0000 C CNN
 F 2 "" H 5900 7050 50  0001 C CNN
@@
 $EndComp
 $Comp
-L power:GND #PWR?
+L power:GND #PWR0117
 U 1 1 61FBEF63
 P 5300 8950
-F 0 "#PWR?" H 5300 8700 50  0001 C CNN
+F 0 "#PWR0117" H 5300 8700 50  0001 C CNN
 F 1 "GND" H 5305 8777 50  0000 C CNN
 F 2 "" H 5300 8950 50  0001 C CNN
@@
 $EndComp
 $Comp
-L power:GND #PWR?
+L power:GND #PWR0118
 U 1 1 61FC7A00
 P 1350 10350
-F 0 "#PWR?" H 1350 10100 50  0001 C CNN
+F 0 "#PWR0118" H 1350 10100 50  0001 C CNN
 F 1 "GND" H 1355 10177 50  0000 C CNN
 F 2 "" H 1350 10350 50  0001 C CNN
@@
 Wire Wire Line
 	4650 8850 4750 8850
-$Comp
-L Device:C_Small C23
-U 1 1 620465DE
-P 6200 8700
-F 0 "C23" H 6292 8746 50  0000 L CNN
-F 1 "100n" H 6292 8655 50  0000 L CNN
-F 2 "Capacitor_SMD:C_1206_3216Metric" H 6200 8700 50  0001 C CNN
-F 3 "~" H 6200 8700 50  0001 C CNN
-	1    6200 8700
-	1    0    0    -1
-$EndComp
 $Comp
 L Device:C_Small C24
@@
 $EndComp
 $Comp
-L power:GND #PWR?
+L power:GND #PWR0119
 U 1 1 620D30F3
 P 8650 6700
-F 0 "#PWR?" H 8650 6450 50  0001 C CNN
+F 0 "#PWR0119" H 8650 6450 50  0001 C CNN
 F 1 "GND" H 8655 6527 50  0000 C CNN
 F 2 "" H 8650 6700 50  0001 C CNN
@@
 F 0 "J21" H 1468 3717 50  0000 C CNN
 F 1 "Conn_01x02" H 1468 3626 50  0000 C CNN
-F 2 "" H 1550 3500 50  0001 C CNN
+F 2 "power_board_for_egs002:conn_5.08" H 1550 3500 50  0001 C CNN
 F 3 "~" H 1550 3500 50  0001 C CNN
 	1    1550 3500
@@
 F 0 "J23" H 1418 5117 50  0000 C CNN
 F 1 "Conn_01x02" H 1418 5026 50  0000 C CNN
-F 2 "" H 1500 4900 50  0001 C CNN
+F 2 "power_board_for_egs002:conn_2.54" H 1500 4900 50  0001 C CNN
 F 3 "~" H 1500 4900 50  0001 C CNN
 	1    1500 4900
@@
 	2850 4900 1700 4900
 $Comp
-L power:GND #PWR?
+L power:GND #PWR0120
 U 1 1 62685F67
 P 3100 5350
-F 0 "#PWR?" H 3100 5100 50  0001 C CNN
+F 0 "#PWR0120" H 3100 5100 50  0001 C CNN
 F 1 "GND" H 3105 5177 50  0000 C CNN
 F 2 "" H 3100 5350 50  0001 C CNN
@@
 $EndComp
 $Comp
-L power:GND #PWR?
+L power:GND #PWR0121
 U 1 1 627ECA89
 P 4250 4550
-F 0 "#PWR?" H 4250 4300 50  0001 C CNN
+F 0 "#PWR0121" H 4250 4300 50  0001 C CNN
 F 1 "GND" H 4255 4377 50  0000 C CNN
 F 2 "" H 4250 4550 50  0001 C CNN

Commit message: continue pcb work
Parts:
- RV21, RV22, RV23: footprint Connector_PinHeader_2.54mm:PinHeader_1x03_P2.54mm_Vertical -> power_board_for_egs002:r_multiturn
Connections:
- net GND: now also J21.1 (Pin_1); no longer J21.2 (Pin_2), R217.1, R218.1, R219.1, R220.1
- net at J22.1 (Pin_1), Q22.3 (S), Q24.3 (S)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: now also J21.2 (Pin_2); no longer J21.1 (Pin_1)
- net at D210.1 (K), D29.2 (A), J23.1 (Pin_1): now also R217.2, R218.2, R219.2, R220.2
- net at D211.2 (A), D212.1 (K), J23.2 (Pin_2): now also R217.1, R218.1, R219.1, R220.1
- new net: D211.1 (K), D29.1 (K), RV21.1
Other:
- moved on the sheet: D210, D211, D212, D29, R217, R218, R219, R220
