File: hardware/power_board_for_egs002/power_supply.sch (KiCad schematic (older format))
At the start: 20 parts, among them J11 +HV_TO_12, J12 +HV_TO_12, J13 HV_TO_12V, J14 12V_TO_5V

Commit message: continue sch update
Parts:
- J11: footprint (none) -> Connector_PinHeader_2.54mm:PinHeader_1x01_P2.54mm_Vertical
- J12: footprint (none) -> Connector_PinHeader_2.54mm:PinHeader_1x01_P2.54mm_
- J13, J14: footprint (none) -> Connector_PinHeader_2.54mm:PinHeader_1x03_P2.54mm_Vertical
Changed lines of the file:
@@
 F 0 "J11" H 2530 1142 50  0000 L CNN
 F 1 "+HV_TO_12" H 2530 1051 50  0000 L CNN
-F 2 "" H 2450 1100 50  0001 C CNN
+F 2 "Connector_PinHeader_2.54mm:PinHeader_1x01_P2.54mm_Vertical" H 2450 1100 50  0001 C CNN
 F 3 "~" H 2450 1100 50  0001 C CNN
 	1    2450 1100
@@
 F 0 "J12" H 2830 1642 50  0000 L CNN
 F 1 "+HV_TO_12" H 2830 1551 50  0000 L CNN
-F 2 "" H 2750 1600 50  0001 C CNN
+F 2 "Connector_PinHeader_2.54mm:PinHeader_1x01_P2.54mm_" H 2750 1600 50  0001 C CNN
 F 3 "~" H 2750 1600 50  0001 C CNN
 	1    2750 1600
@@
 F 0 "J13" V 4014 1362 50  0000 R CNN
 F 1 "HV_TO_12V" V 3923 1362 50  0000 R CNN
-F 2 "" H 4050 1550 50  0001 C CNN
+F 2 "Connector_PinHeader_2.54mm:PinHeader_1x03_P2.54mm_Vertical" H 4050 1550 50  0001 C CNN
 F 3 "~" H 4050 1550 50  0001 C CNN
 	1    4050 1550
@@
 F 0 "J14" V 6214 2562 50  0000 R CNN
 F 1 "12V_TO_5V" V 6123 2562 50  0000 R CNN
-F 2 "" H 6250 2750 50  0001 C CNN
+F 2 "Connector_PinHeader_2.54mm:PinHeader_1x03_P2.54mm_Vertical" H 6250 2750 50  0001 C CNN
 F 3 "~" H 6250 2750 50  0001 C CNN
 	1    6250 2750

Commit message: start adding footprints
Parts:
- C11: renamed from C?; value 470u -> B41858C5477M000; footprint (none) -> Capacitor_THT:CP_Radial_D16.0mm_P7.50mm
- C110, C19: renamed from C?; value C_Small -> 100n; footprint (none) -> Capacitor_SMD:C_1206_3216Metric
- C12, C14, C16: renamed from C?; footprint (none) -> Capacitor_SMD:C_1206_3216Metric
- C13: renamed from C?; footprint (none) -> Capacitor_THT:CP_Radial_D16.0mm_P7.50mm
- C15: renamed from C?; value 470u -> 220u; footprint (none) -> Capacitor_THT:CP_Radial_D16.0mm_P7.50mm
- C17, C18: renamed from C?; value C_Small -> MCKSK050M222J36S; footprint (none) -> Capacitor_THT:CP_Radial_D16.0mm_P7.50mm
- F11, F12, F13: footprint (none) -> power_board_for_egs002:696101000002
- gave numbers to parts that had none: 1
Other:
- moved on the sheet: C110, C18, C19
Changed lines of the file:
@@
 F 0 "F11" H 1300 1035 50  0000 C CNN
 F 1 "Fuse_Small" H 1300 944 50  0000 C CNN
-F 2 "" H 1300 850 50  0001 C CNN
+F 2 "power_board_for_egs002:696101000002" H 1300 850 50  0001 C CNN
 F 3 "~" H 1300 850 50  0001 C CNN
 	1    1300 850
@@
 F 0 "F12" H 1300 2035 50  0000 C CNN
 F 1 "Fuse_Small" H 1300 1944 50  0000 C CNN
-F 2 "" H 1300 1850 50  0001 C CNN
+F 2 "power_board_for_egs002:696101000002" H 1300 1850 50  0001 C CNN
 F 3 "~" H 1300 1850 50  0001 C CNN
 	1    1300 1850
@@
 F 0 "F13" H 1300 3585 50  0000 C CNN
 F 1 "Fuse_Small" H 1300 3494 50  0000 C CNN
-F 2 "" H 1300 3400 50  0001 C CNN
+F 2 "power_board_for_egs002:696101000002" H 1300 3400 50  0001 C CNN
 F 3 "~" H 1300 3400 50  0001 C CNN
 	1    1300 3400
@@
 +12V_RAW
 $Comp
-L Device:C_Small C?
+L Device:C_Small C17
 U 1 1 61B06B90
 P 6700 1050
-F 0 "C?" H 6792 1096 50  0000 L CNN
-F 1 "C_Small" H 6792 1005 50  0000 L CNN
-F 2 "" H 6700 1050 50  0001 C CNN
+F 0 "C17" H 6792 1096 50  0000 L CNN
+F 1 "MCKSK050M222J36S" H 6792 1005 50  0000 L CNN
+F 2 "Capacitor_THT:CP_Radial_D16.0mm_P7.50mm" H 6700 1050 50  0001 C CNN
 F 3 "~" H 6700 1050 50  0001 C CNN
 	1    6700 1050
@@
 $EndComp
 $Comp
-L Device:C_Small C?
+L Device:C_Small C18
 U 1 1 61B0757A
-P 7350 1050
-F 0 "C?" H 7442 1096 50  0000 L CNN
-F 1 "C_Small" H 7442 1005 50  0000 L CNN
-F 2 "" H 7350 1050 50  0001 C CNN
-F 3 "~" H 7350 1050 50  0001 C CNN
-	1    7350 1050
+P 7800 1050
+F 0 "C18" H 7892 1096 50  0000 L CNN
+F 1 "MCKSK050M222J36S" H 7892 1005 50  0000 L CNN
+F 2 "Capacitor_THT:CP_Radial_D16.0mm_P7.50mm" H 7800 1050 50  0001 C CNN
+F 3 "~" H 7800 1050 50  0001 C CNN
+	1    7800 1050
 	1    0    0    -1
 $EndComp
@@
 	4150 1850 4300 1850
 $Comp
-L Device:C_Small C?
+L Device:C_Small C11
 U 1 1 61B0C891
 P 3000 2050
-F 0 "C?" H 3092 2096 50  0000 L CNN
-F 1 "470u" H 3092 2005 50  0000 L CNN
-F 2 "" H 3000 2050 50  0001 C CNN
+F 0 "C11" H 2850 2150 50  0000 L CNN
+F 1 "B41858C5477M000" H 2200 1950 50  0000 L CNN
+F 2 "Capacitor_THT:CP_Radial_D16.0mm_P7.50mm" H 3000 2050 50  0001 C CNN
 F 3 "~" H 3000 2050 50  0001 C CNN
 	1    3000 2050
@@
 $EndComp
 $Comp
-L Device:C_Small C?
+L Device:C_Small C12
 U 1 1 61B0CF2E
 P 3400 2050
-F 0 "C?" H 3492 2096 50  0000 L CNN
+F 0 "C12" H 3492 2096 50  0000 L CNN
 F 1 "100n" H 3492 2005 50  0000 L CNN
-F 2 "" H 3400 2050 50  0001 C CNN
+F 2 "Capacitor_SMD:C_1206_3216Metric" H 3400 2050 50  0001 C CNN
 F 3 "~" H 3400 2050 50  0001 C CNN
 	1    3400 2050
@@
 +12V_REG
 $Comp
-L Device:C_Small C?
+L Device:C_Small C13
 U 1 1 61B125FF
 P 5100 2050
-F 0 "C?" H 5192 2096 50  0000 L CNN
+F 0 "C13" H 5192 2096 50  0000 L CNN
 F 1 "220u" H 5192 2005 50  0000 L CNN
-F 2 "" H 5100 2050 50  0001 C CNN
+F 2 "Capacitor_THT:CP_Radial_D16.0mm_P7.50mm" H 5100 2050 50  0001 C CNN
 F 3 "~" H 5100 2050 50  0001 C CNN
 	1    5100 2050
@@
 $EndComp
 $Comp
-L Device:C_Small C?
+L Device:C_Small C14
 U 1 1 61B12609
 P 5500 2050
-F 0 "C?" H 5592 2096 50  0000 L CNN
+F 0 "C14" H 5592 2096 50  0000 L CNN
 F 1 "100n" H 5592 2005 50  0000 L CNN
-F 2 "" H 5500 2050 50  0001 C CNN
+F 2 "Capacitor_SMD:C_1206_3216Metric" H 5500 2050 50  0001 C CNN
 F 3 "~" H 5500 2050 50  0001 C CNN
 	1    5500 2050
@@
 Connection ~ 6350 3400
 $Comp
-L Device:C_Small C?
+L Device:C_Small C15
 U 1 1 61B21AB9
 P 7550 3600
-F 0 "C?" H 7642 3646 50  0000 L CNN
-F 1 "470u" H 7642 3555 50  0000 L CNN
-F 2 "" H 7550 3600 50  0001 C CNN
+F 0 "C15" H 7642 3646 50  0000 L CNN
+F 1 "220u" H 7642 3555 50  0000 L CNN
+F 2 "Capacitor_THT:CP_Radial_D16.0mm_P7.50mm" H 7550 3600 50  0001 C CNN
 F 3 "~" H 7550 3600 50  0001 C CNN
 	1    7550 3600
@@
 $EndComp
 $Comp
-L Device:C_Small C?
+L Device:C_Small C16
 U 1 1 61B21AC3
 P 7950 3600
-F 0 "C?" H 8042 3646 50  0000 L CNN
+F 0 "C16" H 8042 3646 50  0000 L CNN
 F 1 "100n" H 8042 3555 50  0000 L CNN
-F 2 "" H 7950 3600 50  0001 C CNN
+F 2 "Capacitor_SMD:C_1206_3216Metric" H 7950 3600 50  0001 C CNN
 F 3 "~" H 7950 3600 50  0001 C CNN
 	1    7950 3600
@@
 	7950 3400 10650 3400
 $Comp
-L Diode:1N4007 D?
+L Diode:1N4007 D13
 U 1 1 61B2517A
 P 7000 2500
-F 0 "D?" V 6954 2421 50  0000 R CNN
+F 0 "D13" V 6954 2421 50  0000 R CNN
 F 1 "1N4007" V 7045 2421 50  0000 R CNN
 F 2 "Diode_THT:D_DO-41_SOD81_P10.16mm_Horizontal" H 7000 2325 50  0001 C CNN
@@
 Power supply configuration\n\n1. 3 individual power supplies\n    - remove bridge between J11 and J12\n    - bridge between J13 pin 1 and J13 pin 3\n    - remove the 5V regulator in J14\n\n2. Common +HV and +12V, independent 5V\n    - bridge J11 and J12\n    - bridge between J13 pin 1 and J13 pin 3\n    - remove the 5V regulator in J14\n    - ideally keep +12 as a separate wire to reduce voltage drop\n\n3. Common +HV and 12V, +5V from local regulator:\n    - +HV must not exceed 16V (VGS breakdown)\n    - bridge J11 and J12\n    - bridge between J13 pin 1 and J13 pin 3\n    - add +5V regulator in J14\n    - ideally keep +12 as a separate wire to reduce voltage drop\n\n4. HV only, +12V and +5V from local regulators\n    - bridge J11 and J12\n    - add +12V regulator in J13\n    - add +5V regulator in J14\n\n5. Independent HV and 12V, +5V from local regulator:\n    - remove bridge between J11 and J12\n    - bridge between J13 pin 1 and J13 pin 3\n    - add +5V regulator in J14\n\n6. Independent HV, unregulated +12V, +5V from local regulator\n    - remove bridge between J11 and J12\n    - add +12V regulator in J13\n    - add +5V regulator in J14
 $Comp
-L Device:C_Small C?
+L Device:C_Small C19
 U 1 1 61B48085
-P 7950 1050
-F 0 "C?" H 8042 1096 50  0000 L CNN
-F 1 "C_Small" H 8042 1005 50  0000 L CNN
-F 2 "" H 7950 1050 50  0001 C CNN
-F 3 "~" H 7950 1050 50  0001 C CNN
-	1    7950 1050
-	1    0    0    -1
-$EndComp
-$Comp
-L Device:C_Small C?
+P 9300 1050
+F 0 "C19" H 9392 1096 50  0000 L CNN
+F 1 "100n" H 9392 1005 50  0000 L CNN
+F 2 "Capacitor_SMD:C_1206_3216Metric" H 9300 1050 50  0001 C CNN
+F 3 "~" H 9300 1050 50  0001 C CNN
+	1    9300 1050
+	1    0    0    -1
+$EndComp
+$Comp
+L Device:C_Small C110
 U 1 1 61B4844A
-P 8500 1050
-F 0 "C?" H 8592 1096 50  0000 L CNN
-F 1 "C_Small" H 8592 1005 50  0000 L CNN
-F 2 "" H 8500 1050 50  0001 C CNN
-F 3 "~" H 8500 1050 50  0001 C CNN
-	1    8500 1050
+P 10000 1050
+F 0 "C110" H 10092 1096 50  0000 L CNN
+F 1 "100n" H 10092 1005 50  0000 L CNN
+F 2 "Capacitor_SMD:C_1206_3216Metric" H 10000 1050 50  0001 C CNN
+F 3 "~" H 10000 1050 50  0001 C CNN
+	1    10000 1050
 	1    0    0    -1
 $EndComp
@@
 L power:GND #PWR?
 U 1 1 61B4AC51
-P 7350 1250
-F 0 "#PWR?" H 7350 1000 50  0001 C CNN
-F 1 "GND" H 7355 1077 50  0000 C CNN
-F 2 "" H 7350 1250 50  0001 C CNN
-F 3 "" H 7350 1250 50  0001 C CNN
-	1    7350 1250
+P 7800 1250
+F 0 "#PWR?" H 7800 1000 50  0001 C CNN
+F 1 "GND" H 7805 1077 50  0000 C CNN
+F 2 "" H 7800 1250 50  0001 C CNN
+F 3 "" H 7800 1250 50  0001 C CNN
+	1    7800 1250
 	1    0    0    -1
 $EndComp
@@
 L power:GND #PWR?
 U 1 1 61B4B0FC
-P 7950 1250
-F 0 "#PWR?" H 7950 1000 50  0001 C CNN
-F 1 "GND" H 7955 1077 50  0000 C CNN
-F 2 "" H 7950 1250 50  0001 C CNN
-F 3 "" H 7950 1250 50  0001 C CNN
-	1    7950 1250
+P 9300 1250
+F 0 "#PWR?" H 9300 1000 50  0001 C CNN
+F 1 "GND" H 9305 1077 50  0000 C CNN
+F 2 "" H 9300 1250 50  0001 C CNN
+F 3 "" H 9300 1250 50  0001 C CNN
+	1    9300 1250
 	1    0    0    -1
 $EndComp
@@
 L power:GND #PWR?
 U 1 1 61B4B3AB
-P 8500 1250
-F 0 "#PWR?" H 8500 1000 50  0001 C CNN
-F 1 "GND" H 8505 1077 50  0000 C CNN
-F 2 "" H 8500 1250 50  0001 C CNN
-F 3 "" H 8500 1250 50  0001 C CNN
-	1    8500 1250
-	1    0    0    -1
-$EndComp
-Wire Wire Line
-	8500 1250 8500 1150
-Wire Wire Line
-	7950 1250 7950 1150
-Wire Wire Line
-	7950 850  7950 950
-Connection ~ 7950 850
-Wire Wire Line
-	7950 850  8500 850
-Wire Wire Line
-	8500 950  8500 850
-Connection ~ 8500 850
-Wire Wire Line
-	8500 850  10650 850
-Wire Wire Line
-	7350 950  7350 850
+P 10000 1250
+F 0 "#PWR?" H 10000 1000 50  0001 C CNN
+F 1 "GND" H 10005 1077 50  0000 C CNN
+F 2 "" H 10000 1250 50  0001 C CNN
+F 3 "" H 10000 1250 50  0001 C CNN
+	1    10000 1250
+	1    0    0    -1
+$EndComp
+Wire Wire Line
+	10000 1250 10000 1150
+Wire Wire Line
+	9300 1250 9300 1150
+Wire Wire Line
+	9300 850  9300 950
+Wire Wire Line
+	10000 950  10000 850
+Wire Wire Line
+	7800 950  7800 850
 Wire Wire Line
 	2150 850  6700 850
-Connection ~ 7350 850
-Wire Wire Line
-	7350 850  7950 850
 Wire Wire Line
 	6700 950  6700 850
 Connection ~ 6700 850
 Wire Wire Line
-	6700 850  7350 850
-Wire Wire Line
 	6700 1150 6700 1250
 Wire Wire Line
-	7350 1150 7350 1250
+	7800 1150 7800 1250
+Connection ~ 10000 850
+Wire Wire Line
+	10000 850  10650 850
+Connection ~ 7800 850
+Wire Wire Line
+	7800 850  9300 850
+Wire Wire Line
+	6700 850  7800 850
+Connection ~ 9300 850
+Wire Wire Line
+	9300 850  10000 850
 $EndSCHEMATC

Commit message: continue sch dev
Parts:
- removed F12, F13: Fuse_Small, power_board_for_egs002:696101000002, symbol Device:Fuse_Small
- C11, C13, C15: footprint Capacitor_THT:CP_Radial_D16.0mm_P7.50mm -> Capacitor_THT:CP_Radial_D10.0mm_P5.00mm
- D11, D12, D13: footprint Diode_THT:D_DO-41_SOD81_P10.16mm_Horizontal -> Diode_THT:D_DO-41_SOD81_P5.08mm_Vertical_AnodeUp
- J12: footprint Connector_PinHeader_2.54mm:PinHeader_1x01_P2.54mm_ -> Connector_PinHeader_2.54mm:PinHeader_1x01_P2.54mm_Vertical
- J13, J14: footprint Connector_PinHeader_2.54mm:PinHeader_1x03_P2.54mm_Vertical -> Package_TO_SOT_THT:TO-220-3_Vertical
Connections:
- net +12V_RAW is gone; now on net +12V_IN: C11.1, C12.1, D11.1 (K), D12.1 (K), J13.1 (Pin_1)
- net +5V_OUT is gone; now on net +5V_IN: C15.1, C16.1, D13.2 (A), J14.3 (Pin_3)
Changed lines of the file:
@@
 	1    0    0    -1
 $EndComp
-$Comp
-L Device:Fuse_Small F12
-U 1 1 61AF9B1D
-P 1300 1850
-F 0 "F12" H 1300 2035 50  0000 C CNN
-F 1 "Fuse_Small" H 1300 1944 50  0000 C CNN
-F 2 "power_board_for_egs002:696101000002" H 1300 1850 50  0001 C CNN
-F 3 "~" H 1300 1850 50  0001 C CNN
-	1    1300 1850
-	1    0    0    -1
-$EndComp
-Wire Wire Line
-	1200 1850 950  1850
 Wire Wire Line
 	950  850  1200 850
-$Comp
-L Device:Fuse_Small F13
-U 1 1 61AFB809
-P 1300 3400
-F 0 "F13" H 1300 3585 50  0000 C CNN
-F 1 "Fuse_Small" H 1300 3494 50  0000 C CNN
-F 2 "power_board_for_egs002:696101000002" H 1300 3400 50  0001 C CNN
-F 3 "~" H 1300 3400 50  0001 C CNN
-	1    1300 3400
-	1    0    0    -1
-$EndComp
-Wire Wire Line
-	1200 3400 950  3400
 Wire Wire Line
 	1400 850  2150 850
@@
 F 0 "J12" H 2830 1642 50  0000 L CNN
 F 1 "+HV_TO_12" H 2830 1551 50  0000 L CNN
-F 2 "Connector_PinHeader_2.54mm:PinHeader_1x01_P2.54mm_" H 2750 1600 50  0001 C CNN
+F 2 "Connector_PinHeader_2.54mm:PinHeader_1x01_P2.54mm_Vertical" H 2750 1600 50  0001 C CNN
 F 3 "~" H 2750 1600 50  0001 C CNN
 	1    2750 1600
@@
 $EndComp
 Wire Wire Line
-	1400 1850 2150 1850
-Wire Wire Line
 	2250 1600 2150 1600
 Wire Wire Line
 	2150 1600 2150 1850
-Text Label 1550 1850 0    50   ~ 0
-+12V_RAW
 $Comp
 L Device:C_Small C17
@@
 F 0 "J13" V 4014 1362 50  0000 R CNN
 F 1 "HV_TO_12V" V 3923 1362 50  0000 R CNN
-F 2 "Connector_PinHeader_2.54mm:PinHeader_1x03_P2.54mm_Vertical" H 4050 1550 50  0001 C CNN
+F 2 "Package_TO_SOT_THT:TO-220-3_Vertical" H 4050 1550 50  0001 C CNN
 F 3 "~" H 4050 1550 50  0001 C CNN
 	1    4050 1550
@@
 $EndComp
 $Comp
-L power:GND #PWR?
+L power:GND #PWR0106
 U 1 1 61B09DBD
 P 4050 1950
-F 0 "#PWR?" H 4050 1700 50  0001 C CNN
+F 0 "#PWR0106" H 4050 1700 50  0001 C CNN
 F 1 "GND" H 4055 1777 50  0000 C CNN
 F 2 "" H 4050 1950 50  0001 C CNN
@@
 F 0 "C11" H 2850 2150 50  0000 L CNN
 F 1 "B41858C5477M000" H 2200 1950 50  0000 L CNN
-F 2 "Capacitor_THT:CP_Radial_D16.0mm_P7.50mm" H 3000 2050 50  0001 C CNN
+F 2 "Capacitor_THT:CP_Radial_D10.0mm_P5.00mm" H 3000 2050 50  0001 C CNN
 F 3 "~" H 3000 2050 50  0001 C CNN
 	1    3000 2050
@@
 	3400 1850 3800 1850
 $Comp
-L power:GND #PWR?
+L power:GND #PWR0107
 U 1 1 61B1123F
 P 3000 2250
-F 0 "#PWR?" H 3000 2000 50  0001 C CNN
+F 0 "#PWR0107" H 3000 2000 50  0001 C CNN
 F 1 "GND" H 3005 2077 50  0000 C CNN
 F 2 "" H 3000 2250 50  0001 C CNN
@@
 F 0 "C13" H 5192 2096 50  0000 L CNN
 F 1 "220u" H 5192 2005 50  0000 L CNN
-F 2 "Capacitor_THT:CP_Radial_D16.0mm_P7.50mm" H 5100 2050 50  0001 C CNN
+F 2 "Capacitor_THT:CP_Radial_D10.0mm_P5.00mm" H 5100 2050 50  0001 C CNN
 F 3 "~" H 5100 2050 50  0001 C CNN
 	1    5100 2050
@@
 	5500 1850 5500 1950
 $Comp
-L power:GND #PWR?
+L power:GND #PWR0108
 U 1 1 61B12615
 P 5100 2250
-F 0 "#PWR?" H 5100 2000 50  0001 C CNN
+F 0 "#PWR0108" H 5100 2000 50  0001 C CNN
 F 1 "GND" H 5105 2077 50  0000 C CNN
 F 2 "" H 5100 2250 50  0001 C CNN
@@
 F 0 "D12" H 4050 2334 50  0000 C CNN
 F 1 "1N4007" H 4050 2425 50  0000 C CNN
-F 2 "Diode_THT:D_DO-41_SOD81_P10.16mm_Horizontal" H 4050 2375 50  0001 C CNN
+F 2 "Diode_THT:D_DO-41_SOD81_P5.08mm_Vertical_AnodeUp" H 4050 2375 50  0001 C CNN
 F 3 "http://www.vishay.com/docs/88503/1n4001.pdf" H 4050 2550 50  0001 C CNN
 	1    4050 2550
@@
 F 0 "J14" V 6214 2562 50  0000 R CNN
 F 1 "12V_TO_5V" V 6123 2562 50  0000 R CNN
-F 2 "Connector_PinHeader_2.54mm:PinHeader_1x03_P2.54mm_Vertical" H 6250 2750 50  0001 C CNN
+F 2 "Package_TO_SOT_THT:TO-220-3_Vertical" H 6250 2750 50  0001 C CNN
 F 3 "~" H 6250 2750 50  0001 C CNN
 	1    6250 2750
 	0    -1   -1   0
 $EndComp
-Wire Wire Line
-	1400 3400 6350 3400
 Wire Wire Line
 	6350 3400 6350 2950
@@
 F 0 "C15" H 7642 3646 50  0000 L CNN
 F 1 "220u" H 7642 3555 50  0000 L CNN
-F 2 "Capacitor_THT:CP_Radial_D16.0mm_P7.50mm" H 7550 3600 50  0001 C CNN
+F 2 "Capacitor_THT:CP_Radial_D10.0mm_P5.00mm" H 7550 3600 50  0001 C CNN
 F 3 "~" H 7550 3600 50  0001 C CNN
 	1    7550 3600
@@
 	7950 3400 7950 3500
 $Comp
-L power:GND #PWR?
+L power:GND #PWR0109
 U 1 1 61B21ACF
 P 7550 3800
-F 0 "#PWR?" H 7550 3550 50  0001 C CNN
+F 0 "#PWR0109" H 7550 3550 50  0001 C CNN
 F 1 "GND" H 7555 3627 50  0000 C CNN
 F 2 "" H 7550 3800 50  0001 C CNN
@@
 F 0 "D13" V 6954 2421 50  0000 R CNN
 F 1 "1N4007" V 7045 2421 50  0000 R CNN
-F 2 "Diode_THT:D_DO-41_SOD81_P10.16mm_Horizontal" H 7000 2325 50  0001 C CNN
+F 2 "Diode_THT:D_DO-41_SOD81_P5.08mm_Vertical_AnodeUp" H 7000 2325 50  0001 C CNN
 F 3 "http://www.vishay.com/docs/88503/1n4001.pdf" H 7000 2500 50  0001 C CNN
 	1    7000 2500
@@
 $EndComp
 $Comp
-L power:GND #PWR?
+L power:GND #PWR0110
 U 1 1 61B25B3B
 P 6250 3050
-F 0 "#PWR?" H 6250 2800 50  0001 C CNN
+F 0 "#PWR0110" H 6250 2800 50  0001 C CNN
 F 1 "GND" H 6255 2877 50  0000 C CNN
 F 2 "" H 6250 3050 50  0001 C CNN
@@
 F 0 "D11" H 2400 1384 50  0000 C CNN
 F 1 "1N4007" H 2400 1475 50  0000 C CNN
-F 2 "Diode_THT:D_DO-41_SOD81_P10.16mm_Horizontal" H 2400 1425 50  0001 C CNN
+F 2 "Diode_THT:D_DO-41_SOD81_P5.08mm_Vertical_AnodeUp" H 2400 1425 50  0001 C CNN
 F 3 "http://www.vishay.com/docs/88503/1n4001.pdf" H 2400 1600 50  0001 C CNN
 	1    2400 1600
@@
 $EndComp
 $Comp
-L power:GND #PWR?
+L power:GND #PWR0111
 U 1 1 61B4A0D1
 P 6700 1250
-F 0 "#PWR?" H 6700 1000 50  0001 C CNN
+F 0 "#PWR0111" H 6700 1000 50  0001 C CNN
 F 1 "GND" H 6705 1077 50  0000 C CNN
 F 2 "" H 6700 1250 50  0001 C CNN
@@
 $EndComp
 $Comp
-L power:GND #PWR?
+L power:GND #PWR0112
 U 1 1 61B4AC51
 P 7800 1250
-F 0 "#PWR?" H 7800 1000 50  0001 C CNN
+F 0 "#PWR0112" H 7800 1000 50  0001 C CNN
 F 1 "GND" H 7805 1077 50  0000 C CNN
 F 2 "" H 7800 1250 50  0001 C CNN
@@
 $EndComp
 $Comp
-L power:GND #PWR?
+L power:GND #PWR0113
 U 1 1 61B4B0FC
 P 9300 1250
-F 0 "#PWR?" H 9300 1000 50  0001 C CNN
+F 0 "#PWR0113" H 9300 1000 50  0001 C CNN
 F 1 "GND" H 9305 1077 50  0000 C CNN
 F 2 "" H 9300 1250 50  0001 C CNN
@@
 $EndComp
 $Comp
-L power:GND #PWR?
+L power:GND #PWR0114
 U 1 1 61B4B3AB
 P 10000 1250
-F 0 "#PWR?" H 10000 1000 50  0001 C CNN
+F 0 "#PWR0114" H 10000 1000 50  0001 C CNN
 F 1 "GND" H 10005 1077 50  0000 C CNN
 F 2 "" H 10000 1250 50  0001 C CNN
@@
 Wire Wire Line
 	9300 850  10000 850
+Wire Wire Line
+	950  3400 6350 3400
+Wire Wire Line
+	950  1850 2150 1850
 $EndSCHEMATC

Commit message: continue pcb work
Parts:
- removed F11: Fuse_Small, power_board_for_egs002:696101000002, symbol Device:Fuse_Small
Connections:
- net +HV_OUT is gone; now on net +HV_IN: C110.1, C17.1, C18.1, C19.1, J11.1 (Pin_1)
Changed lines of the file:
@@
 +HV_IN
-$Comp
-L Device:Fuse_Small F11
-U 1 1 61AF9354
-P 1300 850
-F 0 "F11" H 1300 1035 50  0000 C CNN
-F 1 "Fuse_Small" H 1300 944 50  0000 C CNN
-F 2 "power_board_for_egs002:696101000002" H 1300 850 50  0001 C CNN
-F 3 "~" H 1300 850 50  0001 C CNN
-	1    1300 850
-	1    0    0    -1
-$EndComp
-Wire Wire Line
-	950  850  1200 850
-Wire Wire Line
-	1400 850  2150 850
-Text Label 1550 850  0    50   ~ 0
-+HV_RAW
 $Comp
 L Connector_Generic:Conn_01x01 J11
@@
 Wire Wire Line
 	950  1850 2150 1850
+Wire Wire Line
+	950  850  2150 850
 $EndSCHEMATC
