File: hardware/power_board_for_egs002/power_board_for_egs002.kicad_pcb (KiCad board)
At the start: 2 copper layers, 100 x 100 mm, 0 parts

Commit message: continue sch dev
Parts:
- added C11: B41858C5477M000, Capacitor_THT:CP_Radial_D10.0mm_P5.00mm, F.Cu at (53.0, 68.0)
- added C110: 100n, Capacitor_SMD:C_1206_3216Metric, B.Cu at (65.0, 47.0)
- added C12: 100n, Capacitor_SMD:C_1206_3216Metric, B.Cu at (56.0, 70.0)
- added C13: 220u, Capacitor_THT:CP_Radial_D10.0mm_P5.00mm, F.Cu at (47.0, 79.0)
- added C14: 100n, Capacitor_SMD:C_1206_3216Metric, B.Cu at (50.0, 81.4)
- added C15: 220u, Capacitor_THT:CP_Radial_D10.0mm_P5.00mm, F.Cu at (56.0, 91.0)
- added C16: 100n, Capacitor_SMD:C_1206_3216Metric, B.Cu at (59.0, 88.6)
- added C17: MCKSK050M222J36S, Capacitor_THT:CP_Radial_D16.0mm_P7.50mm, F.Cu at (49.0, 45.0)
- added C18: MCKSK050M222J36S, Capacitor_THT:CP_Radial_D16.0mm_P7.50mm, F.Cu at (66.0, 45.0)
- added C19: 100n, Capacitor_SMD:C_1206_3216Metric, B.Cu at (68.0, 41.0)
- added C22: 100n, Capacitor_SMD:C_1206_3216Metric, F.Cu at (157.0, 126.6)
- added C24: 4.7u, Capacitor_THT:CP_Radial_D5.0mm_P2.50mm, F.Cu at (154.0, 120.0)
- added C25: 100n, Capacitor_SMD:C_1206_3216Metric, B.Cu at (139.4, 100.0)
- added C26: 100n, Capacitor_SMD:C_1206_3216Metric, F.Cu at (85.0, 114.0)
- added D11: 1N4007, Diode_THT:D_DO-41_SOD81_P5.08mm_Vertical_AnodeUp, F.Cu at (56.9, 63.0)
- added D12: 1N4007, Diode_THT:D_DO-41_SOD81_P5.08mm_Vertical_AnodeUp, F.Cu at (72.0, 71.0)
- added D13: 1N4007, Diode_THT:D_DO-41_SOD81_P5.08mm_Vertical_AnodeUp, F.Cu at (71.0, 86.0)
- added D21: 1N4148, Diode_THT:D_DO-35_SOD27_P2.54mm_Vertical_AnodeUp, F.Cu at (81.0, 89.0)
- added D210: 1N4148, Diode_THT:D_DO-35_SOD27_P2.54mm_Vertical_AnodeUp, F.Cu at (134.0, 108.5)
- added D211: 1N4148, Diode_THT:D_DO-35_SOD27_P2.54mm_Vertical_AnodeUp, F.Cu at (140.0, 106.0)
- added D212: 1N4148, Diode_THT:D_DO-35_SOD27_P2.54mm_Vertical_AnodeUp, F.Cu at (143.0, 109.0)
- added D213: 1N4007, Diode_THT:D_DO-41_SOD81_P5.08mm_Vertical_AnodeUp, F.Cu at (161.0, 100.0)
- added D214: 1N4007, Diode_THT:D_DO-41_SOD81_P5.08mm_Vertical_AnodeUp, F.Cu at (165.0, 100.0)
- added D215: 1N4007, Diode_THT:D_DO-41_SOD81_P5.08mm_Vertical_AnodeUp, F.Cu at (157.0, 94.9)
- added D216: 1N4007, Diode_THT:D_DO-41_SOD81_P5.08mm_Vertical_AnodeUp, F.Cu at (153.0, 94.9)
- added D22: 1N4148, Diode_THT:D_DO-35_SOD27_P2.54mm_Vertical_AnodeUp, F.Cu at (103.0, 89.0)
- added D23: 1N4148, Diode_THT:D_DO-35_SOD27_P2.54mm_Vertical_AnodeUp, F.Cu at (92.0, 89.0)
- added D24: 1N4148, Diode_THT:D_DO-35_SOD27_P2.54mm_Vertical_AnodeUp, F.Cu at (114.0, 89.0)
- added D25: 1N4148, Diode_THT:D_DO-35_SOD27_P2.54mm_Vertical_AnodeUp, F.Cu at (129.0, 89.0)
- added D26: 1N4148, Diode_THT:D_DO-35_SOD27_P2.54mm_Vertical_AnodeUp, F.Cu at (151.0, 89.0)
- added D27: 1N4148, Diode_THT:D_DO-35_SOD27_P2.54mm_Vertical_AnodeUp, F.Cu at (140.0, 89.0)
- added D28: 1N4148, Diode_THT:D_DO-35_SOD27_P2.54mm_Vertical_AnodeUp, F.Cu at (162.0, 89.0)
- added D29: 1N4148, Diode_THT:D_DO-35_SOD27_P2.54mm_Vertical_AnodeUp, F.Cu at (137.0, 106.0)
- added F11: Fuse_Small, power_board_for_egs002:696101000002, F.Cu at (59.7, 55.0)
- added J1: +HV, power_board_for_egs002:conn_5.08, F.Cu at (42.0, 55.0)
- added J11: +HV_TO_12, Connector_PinHeader_2.54mm:PinHeader_1x01_P2.54mm_Vertical, F.Cu at (71.0, 63.0)
- added J12: +HV_TO_12, Connector_PinHeader_2.54mm:PinHeader_1x01_P2.54mm_Vertical, F.Cu at (66.0, 63.0)
- added J13: HV_TO_12V, Package_TO_SOT_THT:TO-220-3_Vertical, F.Cu at (64.0, 71.0)
- added J14: 12V_TO_5V, Package_TO_SOT_THT:TO-220-3_Vertical, F.Cu at (64.0, 86.0)
- added J2: +12V, power_board_for_egs002:conn_5.08, F.Cu at (42.0, 68.0)
- added J21: Conn_01x02, power_board_for_egs002:conn_5.08, F.Cu at (124.0, 96.0)
- added J22: Conn_01x03, Connector_PinHeader_2.54mm:PinHeader_1x03_P2.54mm_Vertical, F.Cu at (129.0, 96.0)
- added J23: Conn_01x02, power_board_for_egs002:conn_2.54, F.Cu at (137.5, 111.0)
- added J24: HV_SENSE_SELECT_A, Connector_PinHeader_2.54mm:PinHeader_1x03_P2.54mm_Vertical, F.Cu at (167.0, 105.0)
- added J25: HV_SENSE_SELECT_B, Connector_PinHeader_2.54mm:PinHeader_1x03_P2.54mm_Vertical, F.Cu at (161.0, 127.0)
- added J26: Conn_01x02, power_board_for_egs002:conn_2.54, F.Cu at (46.0, 105.0)
- added J3: +5V, power_board_for_egs002:conn_2.54, F.Cu at (40.0, 90.5)
- added J4: BRIGDE_OUT_2, power_board_for_egs002:conn_5.08, F.Cu at (178.0, 48.0)
- added J5: BRIGDE_OUT_1, power_board_for_egs002:conn_5.08, F.Cu at (178.0, 66.0)
- added J6: HV_SENSE, power_board_for_egs002:conn_2.54, F.Cu at (170.0, 98.0)
- added Q21: TK40E06N1, Package_TO_SOT_THT:TO-220-3_Vertical, F.Cu at (81.0, 82.0)
- added Q22: TK40E06N1, Package_TO_SOT_THT:TO-220-3_Vertical, F.Cu at (103.0, 82.0)
- added Q23: TK40E06N1, Package_TO_SOT_THT:TO-220-3_Vertical, F.Cu at (92.0, 82.0)
- added Q24: TK40E06N1, Package_TO_SOT_THT:TO-220-3_Vertical, F.Cu at (114.0, 82.0)
- added Q25: TK40E06N1, Package_TO_SOT_THT:TO-220-3_Vertical, F.Cu at (129.0, 82.0)
- added Q26: TK40E06N1, Package_TO_SOT_THT:TO-220-3_Vertical, F.Cu at (151.0, 82.0)
- added Q27: TK40E06N1, Package_TO_SOT_THT:TO-220-3_Vertical, F.Cu at (140.0, 82.0)
- added Q28: TK40E06N1, Package_TO_SOT_THT:TO-220-3_Vertical, F.Cu at (162.0, 82.0)
- added R21: 5.6, Resistor_SMD:R_1206_3216Metric, B.Cu at (84.0, 88.0)
- added R210: 10k, Resistor_SMD:R_1206_3216Metric, F.Cu at (133.0, 86.0)
- added R211: 5.6, Resistor_SMD:R_1206_3216Metric, B.Cu at (154.0, 88.4)
- added R212: 10k, Resistor_SMD:R_1206_3216Metric, F.Cu at (155.4, 86.0)
- added R213: 5.6, Resistor_SMD:R_1206_3216Metric, B.Cu at (143.0, 88.0)
- added R214: 10k, Resistor_SMD:R_1206_3216Metric, F.Cu at (144.0, 86.0)
- added R215: 5.6, Resistor_SMD:R_1206_3216Metric, B.Cu at (165.0, 88.4)
- added R216: 10k, Resistor_SMD:R_1206_3216Metric, F.Cu at (165.4, 86.0)
- added R217: 10k, Resistor_SMD:R_1206_3216Metric, F.Cu at (134.6, 103.0)
- added R218: 10k, Resistor_SMD:R_1206_3216Metric, F.Cu at (139.4, 103.0)
- added R219: 10k, Resistor_SMD:R_1206_3216Metric, F.Cu at (134.6, 100.0)
- added R22: 10k, Resistor_SMD:R_1206_3216Metric, F.Cu at (85.0, 86.0)
- added R220: 10k, Resistor_SMD:R_1206_3216Metric, F.Cu at (139.4, 100.0)
- added R221: 33k, Resistor_SMD:R_1206_3216Metric, F.Cu at (170.0, 109.4)
- added R222: 33k, Resistor_SMD:R_1206_3216Metric, F.Cu at (167.0, 109.4)
- added R223: 33k, Resistor_SMD:R_1206_3216Metric, F.Cu at (164.0, 109.4)
- added R224: 33k, Resistor_SMD:R_1206_3216Metric, F.Cu at (164.0, 114.4)
- added R225: 33k, Resistor_SMD:R_1206_3216Metric, F.Cu at (167.0, 114.6)
- added R226: 33k, Resistor_SMD:R_1206_3216Metric, F.Cu at (170.0, 114.4)
- added R227: 33k, Resistor_SMD:R_1206_3216Metric, F.Cu at (158.0, 105.0)
- added R228: 33k, Resistor_SMD:R_1206_3216Metric, F.Cu at (158.0, 110.4)
- added R229: 33k, Resistor_SMD:R_1206_3216Metric, F.Cu at (155.0, 109.6)
- added R23: 5.6, Resistor_SMD:R_1206_3216Metric, B.Cu at (106.0, 88.0)
- added R230: 33k, Resistor_SMD:R_1206_3216Metric, F.Cu at (153.0, 104.0)
- added R231: 33k, Resistor_SMD:R_1206_3216Metric, F.Cu at (149.0, 102.4)
- added R232: 33k, Resistor_SMD:R_1206_3216Metric, F.Cu at (149.0, 95.6)
- added R233: 10k, Resistor_SMD:R_1206_3216Metric, F.Cu at (152.0, 109.4)
- added R234: 10k, Resistor_SMD:R_1206_3216Metric, F.Cu at (170.0, 119.4)
- added R235: R_Small, Resistor_SMD:R_1206_3216Metric, B.Cu at (127.0, 98.0)
- added R24: 10k, Resistor_SMD:R_1206_3216Metric, F.Cu at (107.0, 86.0)
- added R25: 5.6, Resistor_SMD:R_1206_3216Metric, B.Cu at (95.0, 88.0)
- added R26: 10k, Resistor_SMD:R_1206_3216Metric, F.Cu at (96.0, 86.0)
- added R27: 5.6, Resistor_SMD:R_1206_3216Metric, B.Cu at (117.0, 88.0)
- added R28: 10k, Resistor_SMD:R_1206_3216Metric, F.Cu at (118.0, 86.0)
- added R29: 5.6, Resistor_SMD:R_1206_3216Metric, B.Cu at (132.0, 88.0)
- added RV21: 100k, Connector_PinHeader_2.54mm:PinHeader_1x03_P2.54mm_Vertical, F.Cu at (136.0, 96.0)
- added RV22: 100k, Connector_PinHeader_2.54mm:PinHeader_1x03_P2.54mm_Vertical, F.Cu at (166.0, 119.0)
- added RV23: 100k, Connector_PinHeader_2.54mm:PinHeader_1x03_P2.54mm_Vertical, F.Cu at (157.0, 115.0)
- added U1: EGS002, power_board_for_egs002:EGS002, F.Cu at (123.0, 120.0)
- added U2: SK68-100SA, power_board_for_egs002:SK68-100SA, F.Cu at (125.0, 55.0)
Other:
- board size 100 x 100 mm -> 150 x 100 mm

Commit message: continue pcb work
Parts:
- removed F11: Fuse_Small, power_board_for_egs002:696101000002
- C25: moved to F.Cu
- RV21, RV22, RV23: footprint Connector_PinHeader_2.54mm:PinHeader_1x03_P2.54mm_Vertical -> power_board_for_egs002:r_multiturn
- moved J6 130.0 mm to (40.0, 99.1)
- moved R230 109.6 mm to (43.5, 106.8)
- moved D214 108.1 mm to (56.9, 102.9)
- moved D213 107.6 mm to (53.4, 102.9)
- moved D216 107.3 mm to (45.7, 97.8)
- moved D215 107.2 mm to (49.8, 97.8)
- moved C24 106.9 mm to (47.2, 113.5)
- moved J24 105.6 mm to (61.4, 102.9), turned to 180 degrees
- moved R221 105.3 mm to (64.7, 107.5), turned to 270 degrees
- moved R227 104.6 mm to (53.4, 107.3)
- moved R234 104.3 mm to (66.0, 111.2), turned to 0 degrees
- moved R231 103.3 mm to (45.8, 106.8)
- moved R226 102.8 mm to (67.5, 107.5)
- moved R222 102.5 mm to (64.7, 102.8)
- moved R228 102.3 mm to (55.8, 107.3), turned to 270 degrees
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Connections:
- C110 pad 1: /PowerSupply/+HV_OUT -> /PowerSupply/+HV_IN
- C17 pad 1: /PowerSupply/+HV_OUT -> /PowerSupply/+HV_IN
- C18 pad 1: /PowerSupply/+HV_OUT -> /PowerSupply/+HV_IN
- C19 pad 1: /PowerSupply/+HV_OUT -> /PowerSupply/+HV_IN
- J11 pad 1: /PowerSupply/+HV_OUT -> /PowerSupply/+HV_IN
- J21 pad 1: Net-(J21-Pad1) -> GND
- J21 pad 2: GND -> Net-(J21-Pad2)
- J22 pad 1: Net-(J21-Pad1) -> Net-(J21-Pad2)
- Q21 pad 2: /PowerSupply/+HV_OUT -> /PowerSupply/+HV_IN
- Q22 pad 3: Net-(J21-Pad1) -> Net-(J21-Pad2)
- Q23 pad 2: /PowerSupply/+HV_OUT -> /PowerSupply/+HV_IN
- Q24 pad 3: Net-(J21-Pad1) -> Net-(J21-Pad2)
- Q25 pad 2: /PowerSupply/+HV_OUT -> /PowerSupply/+HV_IN
- Q26 pad 3: Net-(J21-Pad1) -> Net-(J21-Pad2)
- Q27 pad 2: /PowerSupply/+HV_OUT -> /PowerSupply/+HV_IN
- Q28 pad 3: Net-(J21-Pad1) -> Net-(J21-Pad2)
- R212 pad 1: Net-(J21-Pad1) -> Net-(J21-Pad2)
- R216 pad 1: Net-(J21-Pad1) -> Net-(J21-Pad2)
- R217 pad 1: GND -> Net-(D211-Pad2)
- R217 pad 2: Net-(D211-Pad1) -> Net-(D210-Pad1)
- R218 pad 1: GND -> Net-(D211-Pad2)
- R218 pad 2: Net-(D211-Pad1) -> Net-(D210-Pad1)
- R219 pad 1: GND -> Net-(D211-Pad2)
- R219 pad 2: Net-(D211-Pad1) -> Net-(D210-Pad1)
- R220 pad 1: GND -> Net-(D211-Pad2)
- R220 pad 2: Net-(D211-Pad1) -> Net-(D210-Pad1)
- R235 pad 1: Net-(J21-Pad1) -> Net-(J21-Pad2)
- R24 pad 1: Net-(J21-Pad1) -> Net-(J21-Pad2)
- R28 pad 1: Net-(J21-Pad1) -> Net-(J21-Pad2)
Routing:
- net /PowerBoard/1_VS: track 0.00 -> 96.5 mm, vias 0 -> 2
- net /PowerSupply/+12V_OUT: track 0.00 -> 76.1 mm
- net /PowerSupply/+5V_IN: track 0.00 -> 74.7 mm
- net /PowerBoard/1_HO: track 0.00 -> 71.6 mm, vias 0 -> 2
- net Net-(J21-Pad2): track 0.00 -> 67.8 mm
- net /PowerBoard/2_VS: track 0.00 -> 52.3 mm
- net /PowerBoard/1_LO: track 0.00 -> 48.6 mm
- net /PowerSupply/+12V_IN: track 0.00 -> 47.6 mm
- net /PowerBoard/2_HO: track 0.00 -> 44.3 mm
- net /PowerBoard/2_LO: track 0.00 -> 41.4 mm
- net /PowerBoard/V_FB: track 0.00 -> 34.5 mm
- net Net-(D210-Pad1): track 0.00 -> 32.2 mm
- net Net-(D211-Pad2): track 0.00 -> 31.0 mm
- net Net-(C24-Pad1): track 0.00 -> 21.7 mm
- net /PowerBoard/HV_SENSE_L: track 0.00 -> 21.4 mm
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Other:
- board size 150 x 100 mm -> 150 x 87 mm

Commit message: update layout
Parts:
- moved J11 6.17 mm to (51.4, 47.6)
- moved R235 1.55 mm to (128.1, 97.6)
- moved D13 1.00 mm to (72.0, 84.7)
Routing:
- net Net-(J21-Pad2): track 67.8 -> 36.1 mm
- net /PowerSupply/+5V_IN: track 74.7 -> 92.9 mm
- net /PowerBoard/1_VS: track 96.5 -> 80.5 mm
- net /PowerBoard/2_VS: track 52.3 -> 36.8 mm
- net /PowerSupply/+HV_IN: track 14.7 -> 4.60 mm
- net /PowerSupply/+12V_OUT: track 76.1 -> 78.6 mm
- net GND: vias 0 -> 70
- added copper zone on B.Cu, net /PowerBoard/1_VS
- added copper zone on B.Cu, net /PowerBoard/2_VS
- added copper zone on F.Cu, net /PowerSupply/+HV_IN
- added copper zone on B.Cu, net GND
- added copper zone on F.Cu, net GND
- added copper zone on B.Cu, net Net-(J21-Pad2)
Other:
- board text added: "+"
- board text added: "+12V POWER"
- board text added: "+5V POWER"
- board text added: "BRIDGE POWER"
- board text added: "CT INPUT"
- board text added: "CT OUTPUT"
- board text added: "LIVE"
- board text added: "NEUTRAL"
- board text added: "OUTPUT SENSE H"
- board text added: "SENSE L"
- board text added: "TEMP_FB +5V"
